Commit message: o modelo do robo ja tem as juntas completas. Falta configura-la com porpoçoes do meu corpo!

File: signbot_description/urdf/signbot_full.xacro (robot description, xacro)
@@ -138,5 +138,4 @@
 			middle_length="${LITTLE_MIDDLE_LENGTH}"
 			top_length="${LITTLE_TOP_LENGTH}" />
--->
 <!-- ////////////////// left side /////////////// -->
 <!-- arm -->

File: signbot_final/signbot_f_description/urdf/macros.xacro (robot description, xacro)
@@ -37,8 +37,10 @@
   <property name="THUMB_BOTTOM_LENGTH" value="0.11" />
   <property name="THUMB_TOP_LENGTH" value="${THUMB_RADIUS}" />
+  <property name="THUMB_KNUCKLE_RADIUS" value="0.04" />
 <!-- generic fingers properties -->
   <property name="GENERIC_FINGERS_RADIUS" value="0.05" />
   <property name="GENERIC_FINGERS_X" value="0.027" />
   <property name="INTERVAL_BETWEEN_FINGERS" value="0.01" />
+  <property name="GENERIC_FINGER_KNUCKLE_RADIUS" value="0.03" />
 <!-- index finger properties -->
   <property name="INDEX_BOTTOM_LENGTH" value="0.1" />
@@ -223,7 +225,7 @@
 </xacro:macro>
 <!-- ******************************************************************************************** -->
-<!-- ****************************************** HAND ******************************************** -->
-<!-- ******************************************************************************************** -->
-<xacro:macro name="hand" params="side axis_y_signal">
+<!-- ****************************************** PALM ******************************************** -->
+<!-- ******************************************************************************************** -->
+<xacro:macro name="palm" params="side axis_y_signal">
 <!-- ***************************************** WIRST1 ******************************************* -->
   <xacro:link_shape name="${side}_wirst1_l" color="Blue" mass="${LIGHTWEIGHT}">
@@ -273,3 +275,175 @@
    <xacro:transmission_block joint_name="${side}_wirst3_j"/>
 </xacro:macro>
+<!-- ******************************************************************************************** -->
+<!-- ********************************** THUMB FINGER ******************************************** -->
+<!-- ******************************************************************************************** -->
+<!-- ****************************** BOT KNICKLE ************************************************* -->
+<xacro:macro name="thumb_finger" params="side axis_y_signal lower upper ">
+    <xacro:link_shape name="${side}_bottom_knuckle_thumb_l" color="Blue" mass="${LIGHTWEIGHT}">
+        <origin rpy="0 0 0" xyz="0 0 0"/>
+        <sphere radius="${THUMB_RADIUS}" />
+    </xacro:link_shape>
+    <xacro:gazebo_blue name="{side}_bottom_knuckle_thumb_l" />
+    <joint name="${side}_bottom_knuckle_thumb_j" type="revolute">
+        <parent link="${side}_palm_l"/>
+        <child link="${side}_bottom_knuckle_thumb_l"/>
+        <origin xyz="0 ${axis_y_signal*THUMB_RADIUS} ${(PALM_LENGTH/2)+THUMB_RADIUS+TOLERANCE}" />
+        <axis xyz="1 0 0"/>
+        <limit effort="1000.0" lower="-${lower*(PI/2)}" upper="${upper*(PI/2)}" velocity="0.5"/>
+        <dynamics damping="50" friction="1"/>
+    </joint>
+<!-- ********************************** BOT THUMB ********************************************** -->
+    <xacro:link_shape name="${side}_bottom_thumb_l" color="White" mass="${LIGHTWEIGHT}">
+        <origin rpy="0 0 0" xyz="0 0 ${THUMB_BOTTOM_LENGTH/2}"/>
+        <cylinder radius="${THUMB_RADIUS}" length="${THUMB_BOTTOM_LENGTH}"/>
+    </xacro:link_shape>
+    <xacro:gazebo_white name="{side}_bottom_thumb_l" />
+    <joint name="${side}_knuckle_upper_thumb_j" type="revolute">
+        <parent link="${side}_bottom_knuckle_thumb_l"/>
+        <child link="${side}_bottom_thumb_l"/>
+        <origin xyz="0 0 0"/>
+        <axis xyz="0 1 0"/>
+        <limit effort="1000.0" lower="0" upper="${PI/2}" velocity="0.5"/>
+        <dynamics damping="50" friction="1"/>
+    </joint>
+<!-- *********************************** MIDDLE KNUCKLE ****************************************** -->
+      <xacro:link_shape name="${side}_middle_knuckle_thumb_l" color="Blue" mass="${LIGHTWEIGHT}" >
+          <origin rpy="0 ${PI/2} 0" xyz="0 0 0"/>
+          <cylinder radius="${THUMB_KNUCKLE_RADIUS}" length="${THUMB_RADIUS*2}"/>
+      </xacro:link_shape>
+      <xacro:gazebo_blue name="{side}_middle_thumb_l" />
+      <joint name="${side}_middle_knuckle_thumb_j" type="revolute">
+          <parent link="${side}_bottom_thumb_l"/>
+          <child link="${side}_middle_knuckle_thumb_l"/>
+          <origin xyz="0 0 ${THUMB_BOTTOM_LENGTH+THUMB_KNUCKLE_RADIUS}"/>
+          <axis xyz="1 0 0"/>
+          <limit effort="1000.0" lower="-${lower*(PI/2)}" upper="${upper*(PI/2)}" velocity="0.5"/>
+          <dynamics damping="50" friction="1"/>
+      </joint>
+<!-- ************************************ MIDDLE THUMB ****************************************** -->
+    <xacro:link_shape name="${side}_middle_thumb_l" color="White" mass="${LIGHTWEIGHT}" >
+        <origin rpy="0 0 0" xyz="0 0 ${THUMB_TOP_LENGTH/2}"/>
+        <cylinder radius="${THUMB_RADIUS}" length="${THUMB_TOP_LENGTH}"/>
+    </xacro:link_shape>
+    <xacro:gazebo_white name="{side}_middle_thumb_l" />
+    <joint name="${side}_middle_thumb_j" type="fixed">
+        <parent link="${side}_middle_knuckle_thumb_l"/>
+        <child link="${side}_middle_thumb_l"/>
+        <origin xyz="0 0 ${THUMB_KNUCKLE_RADIUS}"/>
+    </joint>
+<!-- ************************************ TOP THUMB ******************************************** -->
+    <xacro:link_shape name="${side}_top_thumb_l" color="White" mass="${LIGHTWEIGHT}">
+        <origin rpy="0 0 0" xyz="0 0 0"/>
+        <sphere radius="${THUMB_RADIUS}"/>
+    </xacro:link_shape>
+    <xacro:gazebo_white name="{side}_top_thumb_l" />
+    <joint name="${side}_top_thumb_j" type="fixed">
+        <parent link="${side}_middle_thumb_l"/>
+        <child link="${side}_top_thumb_l"/>
+        <origin xyz="0 0 ${THUMB_TOP_LENGTH}"/>
+    </joint>
+<!-- ************************************ TRANSMICION ROS CONTROL ******************************* -->
+   <xacro:transmission_block joint_name="${side}_bottom_knuckle_thumb_j"/>
+   <xacro:transmission_block joint_name="${side}_knuckle_upper_thumb_j"/>
+   <xacro:transmission_block joint_name="${side}_middle_knuckle_thumb_j"/>
+</xacro:macro>
+<!-- ********************************************************************************************* -->
+<!-- ********************************** GENERIC FINGER	******************************************
+      palm -> 0.43 for 4 fingers + 0.01 of interval between fingers
+              finger radius: 0.05
+              0.05*2*4+3*0.01 = 0.43 -->
+<!-- ********************************************************************************************* -->
+<xacro:macro name="generic_finger"
+        params="name side axis_y_signal lower upper ref_point bottom_length middle_length top_length">
+<!-- ***************************************** BOT KNUCKLE *************************************** -->
+    <xacro:link_shape name="${side}_bottom_knuckle_${name}_l" color="Blue" mass="${LIGHTWEIGHT}">
+        <origin rpy="0 0 0" xyz="0 0 0"/>
+        <sphere radius="${GENERIC_FINGERS_RADIUS}" />
+    </xacro:link_shape>
+    <xacro:gazebo_blue name="{side}_bottom_knuckle_${name}_l" />
+    <joint name="${side}_bottom_knuckle_${name}_j" type="revolute">
+        <parent link="${side}_palm_l"/>
+        <child link="${side}_bottom_knuckle_${name}_l"/>
+        <origin xyz="${GENERIC_FINGERS_X} ${axis_y_signal*PALM_HEIGHT} ${ref_point}"/>
+        <axis xyz="0 0 1"/>
+        <limit effort="1000.0" lower="-${lower*(PI/2)}" upper="${upper*(PI/2)}" velocity="0.5"/>
+        <dynamics damping="50" friction="1"/>
+    </joint>
+<!-- ************************************* BOT FINGER ******************************************** -->
+    <xacro:link_shape name="${side}_bottom_${name}_l" color="White" mass="${LIGHTWEIGHT}">
+        <origin rpy="${PI/2} 0 0" xyz="0 ${axis_y_signal*(bottom_length/2)} 0"/>
+        <cylinder radius="${GENERIC_FINGERS_RADIUS}" length="${bottom_length}"/>
+    </xacro:link_shape>
+    <xacro:gazebo_white name="{side}_bottom_${name}_l" />
+    <joint name="${side}_knuckle_upper_${name}_j" type="fixed">
+        <parent link="${side}_bottom_knuckle_${name}_l"/>
+        <child link="${side}_bottom_${name}_l"/>
+        <origin xyz="0 ${axis_y_signal*GENERIC_FINGERS_RADIUS} 0"/>
+    </joint>
+<!-- ***************************************** MIDDLE KNUCKLE ************************************** -->
+  <xacro:link_shape name="${side}_middle_knuckle_${name}_l" color="Blue" mass="${LIGHTWEIGHT}">
+      <origin rpy="0 0 0" xyz="0 0 0"/>
+      <cylinder radius="${GENERIC_FINGER_KNUCKLE_RADIUS}" length="${GENERIC_FINGERS_RADIUS*2}"/>
+  </xacro:link_shape>
+  <xacro:gazebo_blue name="{side}_middle_knuckle_${name}_l" />
+  <joint name="${side}_middle_knuckle_${name}_j" type="revolute">
+      <parent link="${side}_bottom_${name}_l"/>
+      <child link="${side}_middle_knuckle_${name}_l"/>
+      <origin xyz="0 ${axis_y_signal*(bottom_length+GENERIC_FINGER_KNUCKLE_RADIUS)} 0"/>
+      <axis xyz="0 0 1"/>
+  <limit effort="1000.0" lower="-${lower*(PI/2)}" upper="${upper*(PI/2)}" velocity="0.5"/>
+  <dynamics damping="50" friction="1"/>
+  </joint>
+<!-- ***************************************** MIDDLE FINGER ************************************** -->
+    <xacro:link_shape name="${side}_middle_${name}_l" color="White" mass="${LIGHTWEIGHT}">
+        <origin rpy="${PI/2} 0 0" xyz="0 ${axis_y_signal*(middle_length/2)} 0"/>
+        <cylinder radius="${GENERIC_FINGERS_RADIUS}" length="${middle_length}"/>
+    </xacro:link_shape>
+    <xacro:gazebo_white name="{side}_middle_${name}_l" />
+    <joint name="${side}_middle_${name}_j" type="fixed">
+        <parent link="${side}_middle_knuckle_${name}_l"/>
+        <child link="${side}_middle_${name}_l"/>
+        <origin xyz="0 ${axis_y_signal*(GENERIC_FINGER_KNUCKLE_RADIUS)} 0"/>
+    </joint>
+<!-- ***************************************** TOP KNUCKLE **************************************** -->
+    <xacro:link_shape name="${side}_top_knuckle_${name}_l" color="Blue" mass="${LIGHTWEIGHT}">
+        <origin rpy="0 0 0" xyz="0 0 0"/>
+        <cylinder radius="${GENERIC_FINGER_KNUCKLE_RADIUS}" length="${GENERIC_FINGERS_RADIUS*2}"/>
+    </xacro:link_shape>
+    <xacro:gazebo_blue name="{side}_top_knuckle_${name}_l" />
+    <joint name="${side}_top_knuckle_${name}_j" type="revolute">
+        <parent link="${side}_middle_${name}_l"/>
+        <child link="${side}_top_knuckle_${name}_l"/>
+        <origin xyz="0 ${axis_y_signal*(middle_length+GENERIC_FINGER_KNUCKLE_RADIUS)} 0"/>
+        <axis xyz="0 0 1"/>
+        <limit effort="1000.0" lower="-${lower*(PI/2)}" upper="${upper*(PI/2)}" velocity="0.5"/>
+        <dynamics damping="50" friction="1"/>
+    </joint>
+<!-- ******************************************** TOP FINGER ************************************** -->
+    <xacro:link_shape name="${side}_top_${name}_l" color="White" mass="${LIGHTWEIGHT}">
+        <origin rpy="${PI/2} 0 0" xyz="0 ${axis_y_signal*(top_length/2)} 0"/>
+        <cylinder radius="${GENERIC_FINGERS_RADIUS}" length="${top_length}"/>
+    </xacro:link_shape>
+    <xacro:gazebo_white name="{side}_top_${name}_l" />
+    <joint name="${side}_top_${name}_j" type="fixed">
+        <parent link="${side}_top_knuckle_${name}_l"/>
+        <child link="${side}_top_${name}_l"/>
+        <origin xyz="0 ${axis_y_signal*GENERIC_FINGER_KNUCKLE_RADIUS} 0"/>
+    </joint>
+<!-- ****************************************** TOPTOP FINGER ************************************* -->
+    <xacro:link_shape name="${side}_toptop_${name}_l" color="White" mass="${LIGHTWEIGHT}">
+        <origin rpy="0 0 0" xyz="0 0 0"/>
+        <sphere radius="${GENERIC_FINGERS_RADIUS}"/>
+    </xacro:link_shape>
+    <xacro:gazebo_white name="{side}_toptop_${name}_l" />
+    <joint name="${side}_toptop_${name}_j" type="fixed">
+        <parent link="${side}_top_${name}_l"/>
+        <child link="${side}_toptop_${name}_l"/>
+        <origin xyz="0 ${axis_y_signal*GENERIC_FINGERS_RADIUS} 0"/>
+    </joint>
+<!-- ********************************** TRANSMICION ROS CONTROL *********************************** -->
+   <xacro:transmission_block joint_name="${side}_bottom_knuckle_${name}_j"/>
+   <xacro:transmission_block joint_name="${side}_middle_knuckle_${name}_j"/>
+   <xacro:transmission_block joint_name="${side}_top_knuckle_${name}_j"/>
+</xacro:macro>
 </robot>

File: signbot_final/signbot_f_description/urdf/signbot.xacro (robot description, xacro)
@@ -13,21 +13,109 @@
 <!-- ************************** LEG TOSRO AND HEAD ******************************* -->
 <xacro:torso_head parentl_name="base_link" />
-<!-- ****************************** RIGHT SIDE *********************************** -->
-<!-- ********************************** ARM ************************************** -->
+<!-- ****************************************************************************** -->
+<!-- ****************************** RIGHT SIDE ************************************ -->
+<!-- ****************************************************************************** -->
+<!-- ********************************** ARM *************************************** -->
   <xacro:arm side="r"
              axis_y_signal="-1"
              lower="0"
              upper="1" />
-<!-- *********************************** HAND ************************************ -->
-  <xacro:hand side="r"
+<!-- *********************************** PALM ************************************* -->
+  <xacro:palm side="r"
               axis_y_signal="-1" />
-<!-- ****************************** LEFT SIDE ************************************ -->
-<!-- ********************************** ARM ************************************** -->
+<!-- ************************************ THUMB *********************************** -->
+  <xacro:thumb_finger side="r"
+                      axis_y_signal="-1"
+                      lower="0"
+                      upper="1" />
+<!-- **************** FOUR FINGERS (INDEX, MIDDLE, THIRD, LITTLE) ****************** -->
+  <xacro:generic_finger name= "index"
+                        side="r"
+                        axis_y_signal="-1"
+                        lower="0"
+                        upper="1"
+                        ref_point="${(PALM_LENGTH/2)-GENERIC_FINGERS_RADIUS}"
+                        bottom_length="${INDEX_BOTTOM_LENGTH}"
+                        middle_length="${INDEX_MIDDLE_LENGTH}"
+                        top_length="${INDEX_TOP_LENGTH}" />
+  <xacro:generic_finger name= "middle"
+                        side="r"
+                        axis_y_signal="-1"
+                        lower="0"
+                        upper="1"
+                        ref_point="${(PALM_LENGTH/2)-GENERIC_FINGERS_RADIUS*3-INTERVAL_BETWEEN_FINGERS}"
+                        bottom_length="${MIDDLE_BOTTOM_LENGTH}"
+                        middle_length="${MIDDLE_MIDDLE_LENGTH}"
+                        top_length="${MIDDLE_TOP_LENGTH}" />
+  <xacro:generic_finger name= "third"
+                        side="r"
+                        axis_y_signal="-1"
+                        lower="0"
+                        upper="1"
+                        ref_point="${(PALM_LENGTH/2)-GENERIC_FINGERS_RADIUS*5-INTERVAL_BETWEEN_FINGERS*2}"
+                        bottom_length="${THIRD_BOTTOM_LENGTH}"
+                        middle_length="${THIRD_MIDDLE_LENGTH}"
+                        top_length="${THIRD_TOP_LENGTH}" />
+  <xacro:generic_finger name= "little"
+                        side="r"
+                        axis_y_signal="-1"
+                        lower="0"
+                        upper="1"
+                        ref_point="${(PALM_LENGTH/2)-GENERIC_FINGERS_RADIUS*7-INTERVAL_BETWEEN_FINGERS*3}"
+                        bottom_length="${LITTLE_BOTTOM_LENGTH}"
+                        middle_length="${LITTLE_MIDDLE_LENGTH}"
+                        top_length="${LITTLE_TOP_LENGTH}" />
+<!-- ****************************************************************************** -->
+<!-- ****************************** LEFT SIDE ************************************* -->
+<!-- ****************************************************************************** -->
+<!-- ********************************** ARM *************************************** -->
   <xacro:arm side="l"
              axis_y_signal="1"
              lower="1"
              upper="0" />
-<!-- *********************************** HAND ************************************ -->
-  <xacro:hand side="l"
+<!-- *********************************** PALM ************************************* -->
+  <xacro:palm side="l"
               axis_y_signal="1" />
+<!-- ************************************ THUMB *********************************** -->
+  <xacro:thumb_finger side="l"
+                      axis_y_signal="1"
+                      lower="1"
+                      upper="0" />
+<!-- ********************* FOUR FINGERS(INDEX, MIDDLE, THIRD, LITTLE) ************* -->
+  <xacro:generic_finger name= "index"
+                        side="l"
+                        axis_y_signal="1"
+                        lower="1"
+                        upper="0"
+                        ref_point="${(PALM_LENGTH/2)-GENERIC_FINGERS_RADIUS}"
+                        bottom_length="${INDEX_BOTTOM_LENGTH}"
+                        middle_length="${INDEX_MIDDLE_LENGTH}"
+                        top_length="${INDEX_TOP_LENGTH}" />
+  <xacro:generic_finger name= "middle"
+                        side="l"
+                        axis_y_signal="1"
+                        lower="1"
+                        upper="0"
+                        ref_point="${(PALM_LENGTH/2)-GENERIC_FINGERS_RADIUS*3-INTERVAL_BETWEEN_FINGERS}"
+                        bottom_length="${MIDDLE_BOTTOM_LENGTH}"
+                        middle_length="${MIDDLE_MIDDLE_LENGTH}"
+                        top_length="${MIDDLE_TOP_LENGTH}" />
+  <xacro:generic_finger name= "third"
+                        side="l"
+                        axis_y_signal="1"
+                        lower="1"
+                        upper="0"
+                        ref_point="${(PALM_LENGTH/2)-GENERIC_FINGERS_RADIUS*5-INTERVAL_BETWEEN_FINGERS*2}"
+                        bottom_length="${THIRD_BOTTOM_LENGTH}"
+                        middle_length="${THIRD_MIDDLE_LENGTH}"
+                        top_length="${THIRD_TOP_LENGTH}" />
+  <xacro:generic_finger name= "little"
+                        side="l"
+                        axis_y_signal="1"
+                        lower="1"
+                        upper="0"
+                        ref_point="${(PALM_LENGTH/2)-GENERIC_FINGERS_RADIUS*7-INTERVAL_BETWEEN_FINGERS*3}"
+                        bottom_length="${LITTLE_BOTTOM_LENGTH}"
+                        middle_length="${LITTLE_MIDDLE_LENGTH}"
+                        top_length="${LITTLE_TOP_LENGTH}" />
 </robot>
