Commit message: signbot_f_descritpion -> urdf completo ate à palma
ainda precisa de inserir os dedos e acertar os proporçoes

File: signbot_final/signbot_f_description/urdf/macros.xacro (robot description, xacro)
@@ -1,4 +1,4 @@
 <?xml version="1.0"?>
-<robot xmlns:xacro="http:***www.ros.org/wiki/xacro">
+<robot xmlns:xacro="http://www.ros.org/wiki/xacro">
 <xacro:include filename="$(find signbot_f_description)/urdf/signbot.gazebo" />
 <xacro:include filename="$(find signbot_f_description)/urdf/materials.xacro" />
@@ -20,9 +20,13 @@
   <property name="HEAD_RADIUS" value="0.4"/>
 <!-- arm link properties -->
+  <property name="SHOULDER_LENGTH" value="0.1" />
   <property name="ARM_RADIUS" value="0.2" />
-  <property name="ARM_TOP_LENGTH" value="0.6" />
-  <property name="ARM_BOTTOM_LENGTH" value="0.7" />
+  <property name="ARM_LENGTH" value="0.6" />
+  <property name="ELBOW_RADIUS" value="0.15" />
+  <property name="ELBOW_LENGTH" value="${2*ARM_RADIUS}" />
+  <property name="FOREARM_LENGTH" value="0.7" />
 <!-- wrist link properties -->
   <property name="WRIST_RADIUS" value="${ARM_RADIUS}" />
+  <property name="WRIST_LENGTH" value="0.05" />
 <!-- palm link properties -->
   <property name="PALM_DEPTH" value="${WRIST_RADIUS}" />
@@ -144,62 +148,77 @@
 <!-- ****************************************** ARMS ******************************************** -->
 <!-- ******************************************************************************************** -->
-<!-- ********************************************************************************************
-      FAZER UMA NOVA VERSAO, CASO O DA REVOLUÇAO NAO DER CERTO!!!!!!
-      TOMAR ATENÇAO AOS NOMES.
-      SERA PRECISO  INCREMENTAR UM NOVO LINK! PARA O OMBRO TER 3DOF'S
-      ******************************************************************************************* -->
-<!-- ********************************* SHOULDER PAN LINK ****************************************
-  <xacro:link_shape name="${side}_shoulder_link" color="Blue" mass="${LIGHTWEIGHT}">
+<xacro:macro name="arm" params="side axis_y_signal lower upper" >
+<!-- ********************************* SHOULDER1 LINK ******************************************* -->
+  <xacro:link_shape name="${side}_shoulder1_link" color="Blue" mass="${LIGHTWEIGHT}">
+        <origin xyz="0 0 0" rpy="${PI/2} 0 0" />
+         <cylinder radius="${ARM_RADIUS}" length="${SHOULDER_LENGTH}"/>
+  </xacro:link_shape>
+  <xacro:gazebo_blue name="{side}_shoulder1_link" />
+  <joint name="${side}_shoulder1_joint" type="revolute">
+    <parent link="torso_link"/>
+    <child link="${side}_shoulder1_link"/>
+    <origin xyz="0 ${axis_y_signal*((TORSO_LENGTH/2)+(SHOULDER_LENGTH/2))} ${TORSO_HEIGHT-ARM_RADIUS}"/>
+    <axis xyz="0 1 0"/>
+    <limit effort="1000.0" lower="0" upper="${PI/2}" velocity="0.5"/>
+    <dynamics damping="50" friction="1"/>
+  </joint>
+<!-- ********************************* SHOULDER2 LINK **************************************** -->
+  <xacro:link_shape name="${side}_shoulder2_link" color="Blue" mass="${LIGHTWEIGHT}">
         <origin xyz="0 0 0" rpy="0 0 0" />
         <sphere radius="${ARM_RADIUS}"/>
   </xacro:link_shape>
-  <gazebo reference="${side}_shoulder_link">
-    <material>Gazebo/Blue</material>
-  </gazebo>
-  <joint name="${side}_shoulder_joint" type="revolute">
-    <parent link="torso_link"/>
-    <child link="${side}_shoulder_link"/>
-    <origin xyz="0 ${axis_y_signal*((TORSO_LENGTH/2)+ARM_RADIUS)} ${TORSO_HEIGHT-ARM_RADIUS}"/>
-    <axis xyz="0 1 0"/>
-    <limit effort="1000.0" lower="-${PI/2}" upper="${PI/2}" velocity="0.5"/>
-    <dynamics damping="50" friction="1"/>
-  </joint>
-<!-- ****************************************** TOP ARM *****************************************
-  <xacro:link_shape name="${side}_top_arm_link" color="White" mass="${LIGHTWEIGHT}">
-        <origin rpy="${PI/2} 0 0" xyz="0 ${axis_y_signal*(ARM_TOP_LENGTH/2)} 0"/>
-        <cylinder radius="${ARM_RADIUS}" length="${ARM_TOP_LENGTH}"/>
-  </xacro:link_shape>
-  <gazebo reference="${side}_top_arm_link">
-    <material>Gazebo/White</material>
-  </gazebo>
-  <joint name="${side}_top_arm_joint" type="revolute">
-    <parent link="${side}_shoulder_link"/>
-    <child link="${side}_top_arm_link"/>
-    <origin xyz="0 0 0"/>
+  <xacro:gazebo_blue name="{side}_shoulder2_link" />
+  <joint name="${side}_shoulder2_joint" type="revolute">
+    <parent link="${side}_shoulder1_link"/>
+    <child link="${side}_shoulder2_link"/>
+    <origin xyz="0 ${axis_y_signal*((SHOULDER_LENGTH/2)+ARM_RADIUS)} 0"/>
     <axis xyz="0 0 1"/>
     <limit effort="1000.0" lower="${lower*(-1*(PI/2))}" upper="${upper*(PI/2)}" velocity="0.5"/>
     <dynamics damping="50" friction="1"/>
   </joint>
-<!-- ****************************************** BOTTOM ARM **************************************
-  <xacro:link_shape name="${side}_bottom_arm_link" color="White" mass="${LIGHTWEIGHT}">
-         <origin rpy="${PI/2} 0 0" xyz="-${ARM_RADIUS} ${axis_y_signal*(ARM_BOTTOM_LENGTH/2)} 0"/>
-         <cylinder radius="${ARM_RADIUS}" length="${ARM_BOTTOM_LENGTH}"/>
-  </xacro:link_shape>
-  <gazebo reference="${side}_bottom_arm_link">
-    <material>Gazebo/White</material>
-  </gazebo>
-  <joint name="${side}_elbow_joint" type="revolute">
-    <parent link="${side}_top_arm_link"/>
-    <child link="${side}_bottom_arm_link"/>
-    <origin xyz="${ARM_RADIUS} ${axis_y_signal*(ARM_TOP_LENGTH)} 0"/>
+<!-- ****************************************** ARM ****************************************** -->
+  <xacro:link_shape name="${side}_arm_link" color="White" mass="${LIGHTWEIGHT}">
+        <origin rpy="${PI/2} 0 0" xyz="0 ${axis_y_signal*(ARM_LENGTH/2)} 0"/>
+        <cylinder radius="${ARM_RADIUS}" length="${ARM_LENGTH}"/>
+  </xacro:link_shape>
+  <xacro:gazebo_white name="{side}_arm_link" />
+  <joint name="${side}_arm_joint" type="revolute">
+    <parent link="${side}_shoulder2_link"/>
+    <child link="${side}_arm_link"/>
+    <origin xyz="0 0 0"/>
+    <axis xyz="1 0 0"/>
+    <limit effort="1000.0" lower="${(-1)*(PI/2)}" upper="${(PI/2)}" velocity="0.5"/>
+    <dynamics damping="50" friction="1"/>
+  </joint>
+<!-- ****************************************** ELBOW ****************************************** -->
+  <xacro:link_shape name="${side}_elbow_link" color="Blue" mass="${LIGHTWEIGHT}">
+        <origin rpy="0 0 0" xyz="0 0 0"/>
+        <cylinder radius="${ELBOW_RADIUS}" length="${ELBOW_LENGTH}"/>
+  </xacro:link_shape>
+  <xacro:gazebo_blue name="{side}_elbow_link" />
+  <joint name="${side}_elbow1_joint" type="revolute">
+    <parent link="${side}_arm_link"/>
+    <child link="${side}_elbow_link"/>
+    <origin xyz="0 ${axis_y_signal*(ARM_LENGTH+ELBOW_RADIUS)} 0"/>
     <axis xyz="0 0 1"/>
-    <limit effort="1000.0" lower="${lower*(-1)*(PI-0.4)}" upper="${upper*(PI-0.4)}" velocity="0.5"/>
-    <dynamics damping="50" friction="1"/>
-  </joint>
-<!-- ************************************** TRANSMICION ROS CONTROL ****************************
-        <xacro:transmission_block joint_name="${side}_shoulder_joint"/>
-        <xacro:transmission_block joint_name="${side}_top_arm_joint"/>
-        <xacro:transmission_block joint_name="${side}_elbow_joint"/>
--->
+    <limit effort="1000.0" lower="${lower*-1*(PI/2)}" upper="${upper*(PI/2)}" velocity="0.5"/>
+    <dynamics damping="50" friction="1"/>
+  </joint>
+<!-- ****************************************** FOREARM **************************************** -->
+  <xacro:link_shape name="${side}_forearm_link" color="White" mass="${LIGHTWEIGHT}">
+         <origin rpy="${PI/2} 0 0" xyz="0 ${axis_y_signal*(FOREARM_LENGTH/2)} 0"/>
+         <cylinder radius="${ARM_RADIUS}" length="${FOREARM_LENGTH}"/>
+  </xacro:link_shape>
+  <xacro:gazebo_white name="{side}_forearm_link" />
+  <joint name="${side}_elbow2_joint" type="fixed">
+    <parent link="${side}_elbow_link"/>
+    <child link="${side}_forearm_link"/>
+    <origin xyz="0 ${axis_y_signal*(ELBOW_RADIUS)} 0"/>
+  </joint>
+<!-- ************************************** TRANSMICION ROS CONTROL **************************** -->
+          <xacro:transmission_block joint_name="${side}_shoulder1_joint"/>
+          <xacro:transmission_block joint_name="${side}_shoulder2_joint"/>
+          <xacro:transmission_block joint_name="${side}_arm_joint"/>
+          <xacro:transmission_block joint_name="${side}_elbow1_joint"/>
 </xacro:macro>
 <!-- ******************************************************************************************** -->
@@ -207,16 +226,28 @@
 <!-- ******************************************************************************************** -->
 <xacro:macro name="hand" params="side axis_y_signal">
-<!-- ***************************************** WIRST ******************************************** -->
-  <xacro:link_shape name="${side}_wirst_l" color="Blue" mass="${LIGHTWEIGHT}">
+<!-- ***************************************** WIRST1 ******************************************* -->
+  <xacro:link_shape name="${side}_wirst1_l" color="Blue" mass="${LIGHTWEIGHT}">
+        <origin xyz="0 0 0" rpy="${PI/2} 0 0" />
+        <cylinder radius="${WRIST_RADIUS}" length="${WRIST_LENGTH}"/>
+  </xacro:link_shape>
+  <xacro:gazebo_blue name="{side}_wirst1_l" />
+  <joint name="${side}_wirst1_j" type="revolute">
+    <parent link="${side}_forearm_link"/>
+    <child link="${side}_wirst1_l"/>
+    <origin xyz="0 ${axis_y_signal*(FOREARM_LENGTH+(WRIST_LENGTH/2))} 0"/>
+    <axis xyz="0 1 0"/>
+    <limit effort="1000.0" lower="0" upper="${PI/2}" velocity="0.5"/>
+    <dynamics damping="50" friction="1"/>
+  </joint>
+<!-- ***************************************** WIRST2 ******************************************* -->
+  <xacro:link_shape name="${side}_wirst2_l" color="Blue" mass="${LIGHTWEIGHT}">
         <origin xyz="0 0 0" rpy="0 0 0" />
         <sphere radius="${WRIST_RADIUS}"/>
   </xacro:link_shape>
-  <gazebo reference="${side}_wirst_l">
-    <material>Gazebo/Blue</material>
-  </gazebo>
-  <joint name="${side}_wirst_j" type="revolute">
-    <parent link="${side}_bottom_arm_link"/>
-    <child link="${side}_wirst_l"/>
-    <origin xyz="-${ARM_RADIUS} ${axis_y_signal*ARM_BOTTOM_LENGTH} 0"/>
+  <xacro:gazebo_blue name="{side}_wirst2_l" />
+  <joint name="${side}_wirst2_j" type="revolute">
+    <parent link="${side}_wirst1_l"/>
+    <child link="${side}_wirst2_l"/>
+    <origin xyz="0 ${axis_y_signal*(WRIST_LENGTH/2)} 0"/>
     <axis xyz="1 0 0"/>
     <limit effort="1000.0" lower="-${PI/4}" upper="${PI/4}" velocity="0.5"/>
@@ -228,9 +259,7 @@
         <box size="${PALM_DEPTH} ${PALM_LENGTH} ${PALM_HEIGHT}"/>
   </xacro:link_shape>
-  <gazebo reference="${side}_palm_l">
-    <material>Gazebo/White</material>
-  </gazebo>
-  <joint name="${side}_upper_wirst_j" type="revolute">
-    <parent link="${side}_wirst_l"/>
+  <xacro:gazebo_blue name="{side}_palm_l" />
+  <joint name="${side}_wirst3_j" type="revolute">
+    <parent link="${side}_wirst2_l"/>
     <child link="${side}_palm_l"/>
     <origin xyz="0 ${axis_y_signal*0.10} 0"/>
@@ -240,6 +269,7 @@
   </joint>
 <!--************************************** TRANSMICION ROS CONTROL ****************************** -->
-   <xacro:transmission_block joint_name="${side}_wirst_j"/>
-   <xacro:transmission_block joint_name="${side}_upper_wirst_j"/>
+   <xacro:transmission_block joint_name="${side}_wirst1_j"/>
+   <xacro:transmission_block joint_name="${side}_wirst2_j"/>
+   <xacro:transmission_block joint_name="${side}_wirst3_j"/>
 </xacro:macro>
 </robot>

File: signbot_final/signbot_f_description/urdf/signbot.xacro (robot description, xacro)
@@ -14,5 +14,5 @@
 <xacro:torso_head parentl_name="base_link" />
 <!-- ****************************** RIGHT SIDE *********************************** -->
-<!-- ******************************* RIGHT ARM *********************************** -->
+<!-- ********************************** ARM ************************************** -->
   <xacro:arm side="r"
              axis_y_signal="-1"
@@ -20,6 +20,14 @@
              upper="1" />
 <!-- *********************************** HAND ************************************ -->
-  <!--<xacro:hand side="r"
+  <xacro:hand side="r"
               axis_y_signal="-1" />
--->
+<!-- ****************************** LEFT SIDE ************************************ -->
+<!-- ********************************** ARM ************************************** -->
+  <xacro:arm side="l"
+             axis_y_signal="1"
+             lower="1"
+             upper="0" />
+<!-- *********************************** HAND ************************************ -->
+  <xacro:hand side="l"
+              axis_y_signal="1" />
 </robot>

Commit message: Adicionado controladores independentes no projeto final.

File: signbot_final/signbot_f_description/urdf/macros.xacro (robot description, xacro)
@@ -156,5 +156,5 @@
          <cylinder radius="${ARM_RADIUS}" length="${SHOULDER_LENGTH}"/>
   </xacro:link_shape>
-  <xacro:gazebo_blue name="{side}_shoulder1_link" />
+  <xacro:gazebo_blue name="${side}_shoulder1_link" />
   <joint name="${side}_shoulder1_joint" type="revolute">
     <parent link="torso_link"/>
@@ -170,5 +170,5 @@
         <sphere radius="${ARM_RADIUS}"/>
   </xacro:link_shape>
-  <xacro:gazebo_blue name="{side}_shoulder2_link" />
+  <xacro:gazebo_blue name="${side}_shoulder2_link" />
   <joint name="${side}_shoulder2_joint" type="revolute">
     <parent link="${side}_shoulder1_link"/>
@@ -184,5 +184,5 @@
         <cylinder radius="${ARM_RADIUS}" length="${ARM_LENGTH}"/>
   </xacro:link_shape>
-  <xacro:gazebo_white name="{side}_arm_link" />
+  <xacro:gazebo_white name="${side}_arm_link" />
   <joint name="${side}_arm_joint" type="revolute">
     <parent link="${side}_shoulder2_link"/>
@@ -198,5 +198,5 @@
         <cylinder radius="${ELBOW_RADIUS}" length="${ELBOW_LENGTH}"/>
   </xacro:link_shape>
-  <xacro:gazebo_blue name="{side}_elbow_link" />
+  <xacro:gazebo_blue name="${side}_elbow_link" />
   <joint name="${side}_elbow1_joint" type="revolute">
     <parent link="${side}_arm_link"/>
@@ -212,5 +212,5 @@
          <cylinder radius="${ARM_RADIUS}" length="${FOREARM_LENGTH}"/>
   </xacro:link_shape>
-  <xacro:gazebo_white name="{side}_forearm_link" />
+  <xacro:gazebo_white name="${side}_forearm_link" />
   <joint name="${side}_elbow2_joint" type="fixed">
     <parent link="${side}_elbow_link"/>
@@ -233,5 +233,5 @@
         <cylinder radius="${WRIST_RADIUS}" length="${WRIST_LENGTH}"/>
   </xacro:link_shape>
-  <xacro:gazebo_blue name="{side}_wirst1_l" />
+  <xacro:gazebo_blue name="${side}_wirst1_l" />
   <joint name="${side}_wirst1_j" type="revolute">
     <parent link="${side}_forearm_link"/>
@@ -247,5 +247,5 @@
         <sphere radius="${WRIST_RADIUS}"/>
   </xacro:link_shape>
-  <xacro:gazebo_blue name="{side}_wirst2_l" />
+  <xacro:gazebo_blue name="${side}_wirst2_l" />
   <joint name="${side}_wirst2_j" type="revolute">
     <parent link="${side}_wirst1_l"/>
@@ -261,5 +261,5 @@
         <box size="${PALM_DEPTH} ${PALM_LENGTH} ${PALM_HEIGHT}"/>
   </xacro:link_shape>
-  <xacro:gazebo_blue name="{side}_palm_l" />
+  <xacro:gazebo_white name="${side}_palm_l" />
   <joint name="${side}_wirst3_j" type="revolute">
     <parent link="${side}_wirst2_l"/>
@@ -284,6 +284,6 @@
         <sphere radius="${THUMB_RADIUS}" />
     </xacro:link_shape>
-    <xacro:gazebo_blue name="{side}_bottom_knuckle_thumb_l" />
-    <joint name="${side}_bottom_knuckle_thumb_j" type="revolute">
+    <xacro:gazebo_blue name="${side}_bottom_knuckle_thumb_l" />
+    <joint name="${side}_bottom_knuckle1_thumb_j" type="revolute">
         <parent link="${side}_palm_l"/>
         <child link="${side}_bottom_knuckle_thumb_l"/>
@@ -298,6 +298,6 @@
         <cylinder radius="${THUMB_RADIUS}" length="${THUMB_BOTTOM_LENGTH}"/>
     </xacro:link_shape>
-    <xacro:gazebo_white name="{side}_bottom_thumb_l" />
-    <joint name="${side}_knuckle_upper_thumb_j" type="revolute">
+    <xacro:gazebo_white name="${side}_bottom_thumb_l" />
+    <joint name="${side}_bottom_knuckle2_thumb_j" type="revolute">
         <parent link="${side}_bottom_knuckle_thumb_l"/>
         <child link="${side}_bottom_thumb_l"/>
@@ -312,6 +312,6 @@
           <cylinder radius="${THUMB_KNUCKLE_RADIUS}" length="${THUMB_RADIUS*2}"/>
       </xacro:link_shape>
-      <xacro:gazebo_blue name="{side}_middle_thumb_l" />
-      <joint name="${side}_middle_knuckle_thumb_j" type="revolute">
+      <xacro:gazebo_blue name="${side}_middle_knuckle_thumb_l" />
+      <joint name="${side}_top_knuckle_thumb_j" type="revolute">
           <parent link="${side}_bottom_thumb_l"/>
           <child link="${side}_middle_knuckle_thumb_l"/>
@@ -326,5 +326,5 @@
         <cylinder radius="${THUMB_RADIUS}" length="${THUMB_TOP_LENGTH}"/>
     </xacro:link_shape>
-    <xacro:gazebo_white name="{side}_middle_thumb_l" />
+    <xacro:gazebo_white name="${side}_middle_thumb_l" />
     <joint name="${side}_middle_thumb_j" type="fixed">
         <parent link="${side}_middle_knuckle_thumb_l"/>
@@ -337,5 +337,5 @@
         <sphere radius="${THUMB_RADIUS}"/>
     </xacro:link_shape>
-    <xacro:gazebo_white name="{side}_top_thumb_l" />
+    <xacro:gazebo_white name="${side}_top_thumb_l" />
     <joint name="${side}_top_thumb_j" type="fixed">
         <parent link="${side}_middle_thumb_l"/>
@@ -344,7 +344,7 @@
     </joint>
 <!-- ************************************ TRANSMICION ROS CONTROL ******************************* -->
-   <xacro:transmission_block joint_name="${side}_bottom_knuckle_thumb_j"/>
-   <xacro:transmission_block joint_name="${side}_knuckle_upper_thumb_j"/>
-   <xacro:transmission_block joint_name="${side}_middle_knuckle_thumb_j"/>
+   <xacro:transmission_block joint_name="${side}_bottom_knuckle1_thumb_j"/>
+   <xacro:transmission_block joint_name="${side}_bottom_knuckle2_thumb_j"/>
+   <xacro:transmission_block joint_name="${side}_top_knuckle_thumb_j"/>
 </xacro:macro>
 <!-- ********************************************************************************************* -->
@@ -361,5 +361,5 @@
         <sphere radius="${GENERIC_FINGERS_RADIUS}" />
     </xacro:link_shape>
-    <xacro:gazebo_blue name="{side}_bottom_knuckle_${name}_l" />
+    <xacro:gazebo_blue name="${side}_bottom_knuckle_${name}_l" />
     <joint name="${side}_bottom_knuckle_${name}_j" type="revolute">
         <parent link="${side}_palm_l"/>
@@ -375,5 +375,5 @@
         <cylinder radius="${GENERIC_FINGERS_RADIUS}" length="${bottom_length}"/>
     </xacro:link_shape>
-    <xacro:gazebo_white name="{side}_bottom_${name}_l" />
+    <xacro:gazebo_white name="${side}_bottom_${name}_l" />
     <joint name="${side}_knuckle_upper_${name}_j" type="fixed">
         <parent link="${side}_bottom_knuckle_${name}_l"/>
@@ -386,5 +386,5 @@
       <cylinder radius="${GENERIC_FINGER_KNUCKLE_RADIUS}" length="${GENERIC_FINGERS_RADIUS*2}"/>
   </xacro:link_shape>
-  <xacro:gazebo_blue name="{side}_middle_knuckle_${name}_l" />
+  <xacro:gazebo_blue name="${side}_middle_knuckle_${name}_l" />
   <joint name="${side}_middle_knuckle_${name}_j" type="revolute">
       <parent link="${side}_bottom_${name}_l"/>
@@ -400,5 +400,5 @@
         <cylinder radius="${GENERIC_FINGERS_RADIUS}" length="${middle_length}"/>
     </xacro:link_shape>
-    <xacro:gazebo_white name="{side}_middle_${name}_l" />
+    <xacro:gazebo_white name="${side}_middle_${name}_l" />
     <joint name="${side}_middle_${name}_j" type="fixed">
         <parent link="${side}_middle_knuckle_${name}_l"/>
@@ -411,5 +411,5 @@
         <cylinder radius="${GENERIC_FINGER_KNUCKLE_RADIUS}" length="${GENERIC_FINGERS_RADIUS*2}"/>
     </xacro:link_shape>
-    <xacro:gazebo_blue name="{side}_top_knuckle_${name}_l" />
+    <xacro:gazebo_blue name="${side}_top_knuckle_${name}_l" />
     <joint name="${side}_top_knuckle_${name}_j" type="revolute">
         <parent link="${side}_middle_${name}_l"/>
@@ -425,5 +425,5 @@
         <cylinder radius="${GENERIC_FINGERS_RADIUS}" length="${top_length}"/>
     </xacro:link_shape>
-    <xacro:gazebo_white name="{side}_top_${name}_l" />
+    <xacro:gazebo_white name="${side}_top_${name}_l" />
     <joint name="${side}_top_${name}_j" type="fixed">
         <parent link="${side}_top_knuckle_${name}_l"/>
@@ -436,5 +436,5 @@
         <sphere radius="${GENERIC_FINGERS_RADIUS}"/>
     </xacro:link_shape>
-    <xacro:gazebo_white name="{side}_toptop_${name}_l" />
+    <xacro:gazebo_white name="${side}_toptop_${name}_l" />
     <joint name="${side}_toptop_${name}_j" type="fixed">
         <parent link="${side}_top_${name}_l"/>
