Commit message: modelo final do robo com porpoçoes humanas.

File: signbot_final/signbot_f_description/urdf/macros.xacro (robot description, xacro)
@@ -10,52 +10,54 @@
   <property name="HEAVYWEIGHT" value="50" />
   <property name="LIGHTWEIGHT" value="1" />
+<!-- Legs Constants -->
+  <property name="LEG_DEPTH" value=".20" />
+  <property name="LEG_LENGTH" value=".39"/>
+  <property name="LEG_HEIGHT" value=".70"/>
 <!-- Torso Constants -->
-  <property name="TORSO_DEPTH" value="0.6" />
-  <property name="TORSO_LENGTH" value="1.4"/>
-  <property name="TORSO_HEIGHT" value="1.6"/>
+  <property name="TORSO_DEPTH" value=".20" />
+  <property name="TORSO_LENGTH" value=".39"/>
+  <property name="TORSO_HEIGHT" value=".50"/>
 <!-- Neck constants -->
-  <property name="NECK_RADIUS" value="0.2" />
-  <property name="NECK_LENGTH" value="0.2"/>
+  <property name="NECK_RADIUS" value="0.05" />
+  <property name="NECK_LENGTH" value="0.1"/>
 <!-- head constants -->
-  <property name="HEAD_RADIUS" value="0.4"/>
+  <property name="HEAD_RADIUS" value="0.15"/>
 <!-- arm link properties -->
-  <property name="SHOULDER_LENGTH" value="0.1" />
-  <property name="ARM_RADIUS" value="0.2" />
-  <property name="ARM_LENGTH" value="0.6" />
-  <property name="ELBOW_RADIUS" value="0.15" />
+  <property name="SHOULDER_LENGTH" value="0.001" />
+  <property name="ARM_RADIUS" value="0.05" />
+  <property name="ARM_LENGTH" value="${0.20-(ELBOW_RADIUS/2)}" />
+  <property name="ELBOW_RADIUS" value="0.03" />
   <property name="ELBOW_LENGTH" value="${2*ARM_RADIUS}" />
-  <property name="FOREARM_LENGTH" value="0.7" />
+  <property name="FOREARM_LENGTH" value="${0.29-(ELBOW_RADIUS/2)}" />
 <!-- wrist link properties -->
   <property name="WRIST_RADIUS" value="${ARM_RADIUS}" />
-  <property name="WRIST_LENGTH" value="0.05" />
+  <property name="WRIST_LENGTH" value="0.01" />
 <!-- palm link properties -->
-  <property name="PALM_DEPTH" value="${WRIST_RADIUS}" />
-  <property name="PALM_LENGTH" value="0.43"/>
-  <property name="PALM_HEIGHT" value="0.35"/>
+  <property name="PALM_DEPTH" value="0.04" />
+  <property name="PALM_LENGTH" value="0.09"/>
+  <property name="PALM_HEIGHT" value="0.09"/>
+<!-- generic fingers properties -->
+  <property name="GENERIC_FINGERS_RADIUS" value="0.01" />
+  <property name="GENERIC_FINGERS_X" value="0.01" />
+  <property name="INTERVAL_BETWEEN_FINGERS" value="0.003" />
+  <property name="GENERIC_FINGER_KNUCKLE_RADIUS" value="0.007" />
 <!-- thumb finger properties -->
-  <property name="THUMB_RADIUS" value="0.06" />
-  <property name="THUMB_BOTTOM_LENGTH" value="0.11" />
-  <property name="THUMB_TOP_LENGTH" value="${THUMB_RADIUS}" />
-  <property name="THUMB_KNUCKLE_RADIUS" value="0.04" />
-<!-- generic fingers properties -->
-  <property name="GENERIC_FINGERS_RADIUS" value="0.05" />
-  <property name="GENERIC_FINGERS_X" value="0.027" />
-  <property name="INTERVAL_BETWEEN_FINGERS" value="0.01" />
-  <property name="GENERIC_FINGER_KNUCKLE_RADIUS" value="0.03" />
+  <property name="THUMB_BOTTOM_LENGTH" value="0.03" />
+  <property name="THUMB_TOP_LENGTH" value="${GENERIC_FINGERS_RADIUS}" />
 <!-- index finger properties -->
-  <property name="INDEX_BOTTOM_LENGTH" value="0.1" />
-  <property name="INDEX_MIDDLE_LENGTH" value="0.09" />
+  <property name="INDEX_BOTTOM_LENGTH" value="0.03" />
+  <property name="INDEX_MIDDLE_LENGTH" value="0.02" />
   <property name="INDEX_TOP_LENGTH" value="${GENERIC_FINGERS_RADIUS}" />
 <!--  middle finger properties  -->
-  <property name="MIDDLE_BOTTOM_LENGTH" value="0.12" />
-  <property name="MIDDLE_MIDDLE_LENGTH" value="0.11" />
+  <property name="MIDDLE_BOTTOM_LENGTH" value="0.04" />
+  <property name="MIDDLE_MIDDLE_LENGTH" value="0.03" />
   <property name="MIDDLE_TOP_LENGTH" value="${GENERIC_FINGERS_RADIUS}" />
 <!--  third finger properties  -->
-  <property name="THIRD_BOTTOM_LENGTH" value="0.1" />
-  <property name="THIRD_MIDDLE_LENGTH" value="0.1" />
+  <property name="THIRD_BOTTOM_LENGTH" value="0.035" />
+  <property name="THIRD_MIDDLE_LENGTH" value="0.02" />
   <property name="THIRD_TOP_LENGTH" value="${GENERIC_FINGERS_RADIUS}" />
 <!--  little finger properties  -->
-  <property name="LITTLE_BOTTOM_LENGTH" value="0.075" />
-  <property name="LITTLE_MIDDLE_LENGTH" value="0.075" />
+  <property name="LITTLE_BOTTOM_LENGTH" value="0.02" />
+  <property name="LITTLE_MIDDLE_LENGTH" value="0.01" />
   <property name="LITTLE_TOP_LENGTH" value="${GENERIC_FINGERS_RADIUS}" />
 <!-- ******************************************************************************************** -->
@@ -109,11 +111,11 @@
   </joint>
   <xacro:link_shape name="legs_link" color="Black"  mass="${HEAVYWEIGHT}" >
-                    <origin xyz="0 0 ${TORSO_HEIGHT/2}" rpy="0 0 0" />
-                    <box size="${TORSO_DEPTH} ${TORSO_LENGTH} ${TORSO_HEIGHT}" />
+                    <origin xyz="0 0 ${LEG_HEIGHT/2}" rpy="0 0 0" />
+                    <box size="${LEG_DEPTH} ${LEG_LENGTH} ${LEG_HEIGHT}" />
   </xacro:link_shape>
   <xacro:gazebo_black name="legs_link" />
   <!-- ************************************ TORSO LINK ****************************************** -->
   <joint name="waist_joint" type="fixed">
-    <origin xyz="0 0 ${TORSO_HEIGHT}" rpy="0 0 0" />
+    <origin xyz="0 0 ${LEG_HEIGHT}" rpy="0 0 0" />
     <parent link="legs_link"/>
     <child link="torso_link"/>
@@ -258,5 +260,5 @@
 <!-- ****************************************** PALM LINK *************************************** -->
   <xacro:link_shape name="${side}_palm_l" color="White" mass="${LIGHTWEIGHT}">
-        <origin rpy="${PI/2} 0 0" xyz="0 ${axis_y_signal*0.17} 0 "/>
+        <origin rpy="${PI/2} 0 0" xyz="0 ${axis_y_signal*PALM_LENGTH/2} 0 "/>
         <box size="${PALM_DEPTH} ${PALM_LENGTH} ${PALM_HEIGHT}"/>
   </xacro:link_shape>
@@ -265,5 +267,5 @@
     <parent link="${side}_wirst2_l"/>
     <child link="${side}_palm_l"/>
-    <origin xyz="0 ${axis_y_signal*0.10} 0"/>
+    <origin xyz="0 ${axis_y_signal*WRIST_RADIUS} 0"/>
     <axis xyz="0 0 1"/>
     <limit effort="1000.0" lower="-${PI/4}" upper="${PI/4}" velocity="0.5"/>
@@ -282,5 +284,5 @@
     <xacro:link_shape name="${side}_bottom_knuckle_thumb_l" color="Blue" mass="${LIGHTWEIGHT}">
         <origin rpy="0 0 0" xyz="0 0 0"/>
-        <sphere radius="${THUMB_RADIUS}" />
+        <sphere radius="${GENERIC_FINGERS_RADIUS}" />
     </xacro:link_shape>
     <xacro:gazebo_blue name="${side}_bottom_knuckle_thumb_l" />
@@ -288,5 +290,5 @@
         <parent link="${side}_palm_l"/>
         <child link="${side}_bottom_knuckle_thumb_l"/>
-        <origin xyz="0 ${axis_y_signal*THUMB_RADIUS} ${(PALM_LENGTH/2)+THUMB_RADIUS+TOLERANCE}" />
+        <origin xyz="0 ${axis_y_signal*GENERIC_FINGERS_RADIUS} ${(PALM_LENGTH/2)+GENERIC_FINGERS_RADIUS+TOLERANCE}" />
         <axis xyz="1 0 0"/>
         <limit effort="1000.0" lower="-${lower*(PI/2)}" upper="${upper*(PI/2)}" velocity="0.5"/>
@@ -296,5 +298,5 @@
     <xacro:link_shape name="${side}_bottom_thumb_l" color="White" mass="${LIGHTWEIGHT}">
         <origin rpy="0 0 0" xyz="0 0 ${THUMB_BOTTOM_LENGTH/2}"/>
-        <cylinder radius="${THUMB_RADIUS}" length="${THUMB_BOTTOM_LENGTH}"/>
+        <cylinder radius="${GENERIC_FINGERS_RADIUS}" length="${THUMB_BOTTOM_LENGTH}"/>
     </xacro:link_shape>
     <xacro:gazebo_white name="${side}_bottom_thumb_l" />
@@ -310,5 +312,5 @@
       <xacro:link_shape name="${side}_middle_knuckle_thumb_l" color="Blue" mass="${LIGHTWEIGHT}" >
           <origin rpy="0 ${PI/2} 0" xyz="0 0 0"/>
-          <cylinder radius="${THUMB_KNUCKLE_RADIUS}" length="${THUMB_RADIUS*2}"/>
+          <cylinder radius="${GENERIC_FINGER_KNUCKLE_RADIUS}" length="${GENERIC_FINGERS_RADIUS*2}"/>
       </xacro:link_shape>
       <xacro:gazebo_blue name="${side}_middle_knuckle_thumb_l" />
@@ -316,5 +318,5 @@
           <parent link="${side}_bottom_thumb_l"/>
           <child link="${side}_middle_knuckle_thumb_l"/>
-          <origin xyz="0 0 ${THUMB_BOTTOM_LENGTH+THUMB_KNUCKLE_RADIUS}"/>
+          <origin xyz="0 0 ${THUMB_BOTTOM_LENGTH+GENERIC_FINGER_KNUCKLE_RADIUS}"/>
           <axis xyz="1 0 0"/>
           <limit effort="1000.0" lower="-${lower*(PI/2)}" upper="${upper*(PI/2)}" velocity="0.5"/>
@@ -324,5 +326,5 @@
     <xacro:link_shape name="${side}_middle_thumb_l" color="White" mass="${LIGHTWEIGHT}" >
         <origin rpy="0 0 0" xyz="0 0 ${THUMB_TOP_LENGTH/2}"/>
-        <cylinder radius="${THUMB_RADIUS}" length="${THUMB_TOP_LENGTH}"/>
+        <cylinder radius="${GENERIC_FINGERS_RADIUS}" length="${THUMB_TOP_LENGTH}"/>
     </xacro:link_shape>
     <xacro:gazebo_white name="${side}_middle_thumb_l" />
@@ -330,10 +332,10 @@
         <parent link="${side}_middle_knuckle_thumb_l"/>
         <child link="${side}_middle_thumb_l"/>
-        <origin xyz="0 0 ${THUMB_KNUCKLE_RADIUS}"/>
+        <origin xyz="0 0 ${GENERIC_FINGER_KNUCKLE_RADIUS}"/>
     </joint>
 <!-- ************************************ TOP THUMB ******************************************** -->
     <xacro:link_shape name="${side}_top_thumb_l" color="White" mass="${LIGHTWEIGHT}">
         <origin rpy="0 0 0" xyz="0 0 0"/>
-        <sphere radius="${THUMB_RADIUS}"/>
+        <sphere radius="${GENERIC_FINGERS_RADIUS}"/>
     </xacro:link_shape>
     <xacro:gazebo_white name="${side}_top_thumb_l" />

File: signbot_final/signbot_f_description/urdf/signbot.xacro (robot description, xacro)
@@ -8,5 +8,5 @@
 <xacro:link_shape name="base_link" color="Black"  mass="${HEAVYWEIGHT}" >
                   <origin xyz="0 0 0" rpy="0 0 0" />
-                  <box size="3 3 0.01" />
+                  <box size="1 1 0.01" />
 </xacro:link_shape>
 <xacro:gazebo_black name="base_link" />
@@ -44,5 +44,5 @@
                         lower="0"
                         upper="1"
-                        ref_point="${(PALM_LENGTH/2)-GENERIC_FINGERS_RADIUS*3-INTERVAL_BETWEEN_FINGERS}"
+                        ref_point="${(PALM_LENGTH/2)-(GENERIC_FINGERS_RADIUS*2)-INTERVAL_BETWEEN_FINGERS-GENERIC_FINGERS_RADIUS}"
                         bottom_length="${MIDDLE_BOTTOM_LENGTH}"
                         middle_length="${MIDDLE_MIDDLE_LENGTH}"
@@ -53,5 +53,5 @@
                         lower="0"
                         upper="1"
-                        ref_point="${(PALM_LENGTH/2)-GENERIC_FINGERS_RADIUS*5-INTERVAL_BETWEEN_FINGERS*2}"
+                        ref_point="${(-PALM_LENGTH/2)+(GENERIC_FINGERS_RADIUS*2)+INTERVAL_BETWEEN_FINGERS+GENERIC_FINGERS_RADIUS}"
                         bottom_length="${THIRD_BOTTOM_LENGTH}"
                         middle_length="${THIRD_MIDDLE_LENGTH}"
@@ -62,5 +62,5 @@
                         lower="0"
                         upper="1"
-                        ref_point="${(PALM_LENGTH/2)-GENERIC_FINGERS_RADIUS*7-INTERVAL_BETWEEN_FINGERS*3}"
+                        ref_point="${(-PALM_LENGTH/2)+GENERIC_FINGERS_RADIUS}"
                         bottom_length="${LITTLE_BOTTOM_LENGTH}"
                         middle_length="${LITTLE_MIDDLE_LENGTH}"

Commit message: terminado o body_controller.launch e yaml

File: signbot_final/signbot_f_description/urdf/macros.xacro (robot description, xacro)
@@ -195,14 +195,28 @@
     <dynamics damping="50" friction="1"/>
   </joint>
-<!-- ****************************************** ELBOW ****************************************** -->
-  <xacro:link_shape name="${side}_elbow_link" color="Blue" mass="${LIGHTWEIGHT}">
-        <origin rpy="0 0 0" xyz="0 0 0"/>
-        <cylinder radius="${ELBOW_RADIUS}" length="${ELBOW_LENGTH}"/>
-  </xacro:link_shape>
-  <xacro:gazebo_blue name="${side}_elbow_link" />
+<!-- ****************************************** ELBOW1 ****************************************** -->
+  <xacro:link_shape name="${side}_elbow1_link" color="Blue" mass="${LIGHTWEIGHT}">
+        <origin xyz="0 0 0" rpy="${PI/2} 0 0" />
+         <cylinder radius="${ARM_RADIUS}" length="${SHOULDER_LENGTH}"/>
+  </xacro:link_shape>
+  <xacro:gazebo_blue name="${side}_elbow1_link" />
   <joint name="${side}_elbow1_joint" type="revolute">
     <parent link="${side}_arm_link"/>
-    <child link="${side}_elbow_link"/>
-    <origin xyz="0 ${axis_y_signal*(ARM_LENGTH+ELBOW_RADIUS)} 0"/>
+    <child link="${side}_elbow1_link"/>
+    <origin xyz="0 ${axis_y_signal*(ARM_LENGTH+(SHOULDER_LENGTH/2))} 0"/>
+    <axis xyz="0 1 0"/>
+    <limit effort="1000.0" lower="${-1*(PI/2)}" upper="${(PI/2)}" velocity="0.5"/>
+    <dynamics damping="50" friction="1"/>
+  </joint>
+<!-- ****************************************** ELBOW2 ****************************************** -->
+  <xacro:link_shape name="${side}_elbow2_link" color="Blue" mass="${LIGHTWEIGHT}">
+        <origin rpy="0 0 0" xyz="0 0 0"/>
+        <cylinder radius="${ELBOW_RADIUS}" length="${ELBOW_LENGTH}"/>
+  </xacro:link_shape>
+  <xacro:gazebo_blue name="${side}_elbow2_link" />
+  <joint name="${side}_elbow2_joint" type="revolute">
+    <parent link="${side}_elbow1_link"/>
+    <child link="${side}_elbow2_link"/>
+    <origin xyz="0 ${axis_y_signal*((SHOULDER_LENGTH/2)+ELBOW_RADIUS)} 0"/>
     <axis xyz="0 0 1"/>
     <limit effort="1000.0" lower="${lower*-1*(PI/2)}" upper="${upper*(PI/2)}" velocity="0.5"/>
@@ -215,6 +229,6 @@
   </xacro:link_shape>
   <xacro:gazebo_white name="${side}_forearm_link" />
-  <joint name="${side}_elbow2_joint" type="fixed">
-    <parent link="${side}_elbow_link"/>
+  <joint name="${side}_elbow3_joint" type="fixed">
+    <parent link="${side}_elbow2_link"/>
     <child link="${side}_forearm_link"/>
     <origin xyz="0 ${axis_y_signal*(ELBOW_RADIUS)} 0"/>
@@ -225,4 +239,5 @@
           <xacro:transmission_block joint_name="${side}_arm_joint"/>
           <xacro:transmission_block joint_name="${side}_elbow1_joint"/>
+          <xacro:transmission_block joint_name="${side}_elbow2_joint"/>
 </xacro:macro>
 <!-- ******************************************************************************************** -->
